Commit message: FInished LV3.

File: src/mob_rob_description/urdf/lv3_mob_rob.urdf (robot description, URDF)
Before this commit: robot mob_rob, 8 links, 7 joints
Links:
- link back_left_wheel: mass 0.1 -> 0.5
- link back_right_wheel: mass 0.1 -> 0.5
- link base_link: mass 1.0 -> 5.0
- link front_left_wheel: mass 0.1 -> 0.5
- link front_right_wheel: mass 0.1 -> 0.5
