Commit message: Finished lv5

File: src/rob_manip_description/urdf/rob_manip.urdf (robot description, URDF)
Before this commit: robot rob_manip, 8 links, 7 joints
Links:
- link forearm_roll_link: geometry collision cylinder length=0.01 radius=0.01; visual cylinder length=0.01 radius=0.01
- link wrist_roll_link: geometry collision cylinder length=0.01 radius=0.01; visual cylinder length=0.01 radius=0.01

Commit message: Revert "Finished lv5"
This reverts commit 94effec79827cf802e502906b2561f27d29a3b82.

File: src/rob_manip_description/urdf/rob_manip.urdf (robot description, URDF)
Before this commit: robot rob_manip, 8 links, 7 joints
Links:
- link forearm_roll_link: geometry visual cylinder length=0.01 radius=0.01
- link wrist_roll_link: geometry visual cylinder length=0.01 radius=0.01

Commit message: LV5 - MoveIt konfiguracija, bringup i control paketi

File: src/rob_manip_description/urdf/rob_manip.urdf (robot description, URDF)
Before this commit: robot rob_manip, 8 links, 7 joints
Links:
- link forearm_roll_link: geometry collision cylinder length=0.01 radius=0.01; visual cylinder length=0.01 radius=0.01
- link hand: mass 1.0 -> 0.5
- link wrist_roll_link: geometry collision cylinder length=0.01 radius=0.01; visual cylinder length=0.01 radius=0.01
Joints:
- joint elbow: limit (none) -> lower=-3.14 upper=3.14 effort=100.0 velocity=3.14; type continuous -> revolute
- joint forearm_roll: limit (none) -> lower=-3.14 upper=3.14 effort=100.0 velocity=3.14; type continuous -> revolute
- joint hand_roll: limit (none) -> lower=-3.14 upper=3.14 effort=100.0 velocity=3.14; type continuous -> revolute
- joint hip: limit (none) -> lower=-3.14 upper=3.14 effort=100.0 velocity=3.14; type continuous -> revolute
- joint shoulder: limit (none) -> lower=-3.14 upper=3.14 effort=100.0 velocity=3.14; type continuous -> revolute
- joint wrist: limit (none) -> lower=-3.14 upper=3.14 effort=100.0 velocity=3.14; type continuous -> revolute
